File: midi_cv_gate_v1.kicad_pcb (KiCad board)
At the start: 2 copper layers, 195 x 100 mm, 330 parts, among them J1 Conn_02x05_Odd_Even, J10 CV_I, J11 CV_J, J12 CV_K, J13 CV_L, J14 CV_M, J15 CV_N, J16 CV_O, J17 CV_P, J18 GATE_A, J19 GATE_B, J2 CV_A, J20 GATE_C, J21 GATE_D, J22 GATE_E, J23 GATE_F, J24 GATE_G, J25 GATE_H, J26 GATE_I, J27 GATE_J, J28 GATE_K, J29 GATE_L, J3 CV_B, J30 GATE_M, J31 GATE_N, J32 GATE_O, J33 GATE_P, J34 Conn_01x10, J35 Conn_01x10, J36 Conn_01x20, J37 Conn_01x20, J39 MIDI OUT, J4 CV_C, J41 MIDI IN, J42 Conn_01x20, J43 Conn_01x20, J5 CV_D, J6 CV_E, J7 CV_F, J8 CV_G, J9 CV_H, Q1 2N3906, Q10 2N3906, Q11 2N3906, Q12 2N3906, Q13 2N3906, Q14 2N3906, Q15 2N3906, Q16 2N3906, Q17 2N3906, Q18 2N3906, Q2 2N3906, Q3 2N3906, Q4 2N3906, Q5 2N3906, Q6 2N3906, Q7 2N3906, Q8 2N3906, Q9 2N3906, SW1 SW_SPST, U1 LM7805_TO220, U10 74HC595, U11 74HC595, U12 LM358, U13 LM358, U14 LM358, U15 LM358, U16 LM358, U17 LM358, U18 LM358, U19 LM358, U2 MCP4922-ESL, U20 LM358, U21 LM358, U22 LM358, U23 LM358, U24 LM358, U25 LM358, U26 LM358, U27 LM358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

Commit message: Replace soic-14 with dip 14 for DACs, add pulldowns on opamp inputs
Parts:
- added H7: MountingHole_Pad, MountingHole:MountingHole_3.2mm_M3_ISO7380_Pad_TopBottom, F.Cu at (54.0, 146.0)
- added H8: MountingHole_Pad, MountingHole:MountingHole_3.2mm_M3_ISO7380_Pad_TopBottom, F.Cu at (159.0, 146.0)
- added R106: 100k, Resistor_SMD:R_1206_3216Metric_Pad1.30x1.75mm_HandSolder, F.Cu at (233.1, 66.3)
- added R164: 100k, Resistor_SMD:R_1206_3216Metric_Pad1.30x1.75mm_HandSolder, F.Cu at (219.8, 72.2)
- added R165: 100k, Resistor_SMD:R_1206_3216Metric_Pad1.30x1.75mm_HandSolder, F.Cu at (233.1, 78.6)
- added R166: 100k, Resistor_SMD:R_1206_3216Metric_Pad1.30x1.75mm_HandSolder, F.Cu at (219.8, 84.5)
- added R167: 100k, Resistor_SMD:R_1206_3216Metric_Pad1.30x1.75mm_HandSolder, F.Cu at (233.1, 91.0)
- added R168: 100k, Resistor_SMD:R_1206_3216Metric_Pad1.30x1.75mm_HandSolder, F.Cu at (219.8, 96.8)
- added R169: 100k, Resistor_SMD:R_1206_3216Metric_Pad1.30x1.75mm_HandSolder, F.Cu at (233.1, 103.3)
- added R170: 100k, Resistor_SMD:R_1206_3216Metric_Pad1.30x1.75mm_HandSolder, F.Cu at (219.8, 109.2)
- added R171: 100k, Resistor_SMD:R_1206_3216Metric_Pad1.30x1.75mm_HandSolder, F.Cu at (233.1, 115.7)
- added R172: 100k, Resistor_SMD:R_1206_3216Metric_Pad1.30x1.75mm_HandSolder, F.Cu at (219.8, 121.5)
- added R173: 100k, Resistor_SMD:R_1206_3216Metric_Pad1.30x1.75mm_HandSolder, F.Cu at (233.1, 128.0)
- added R174: 100k, Resistor_SMD:R_1206_3216Metric_Pad1.30x1.75mm_HandSolder, F.Cu at (219.8, 133.8)
- added R175: 100k, Resistor_SMD:R_1206_3216Metric_Pad1.30x1.75mm_HandSolder, F.Cu at (233.1, 140.3)
- added R176: 100k, Resistor_SMD:R_1206_3216Metric_Pad1.30x1.75mm_HandSolder, F.Cu at (219.8, 146.2)
- added R177: 100k, Resistor_SMD:R_1206_3216Metric_Pad1.30x1.75mm_HandSolder, F.Cu at (180.2, 57.8)
- added R178: 100k, Resistor_SMD:R_1206_3216Metric_Pad1.30x1.75mm_HandSolder, F.Cu at (190.9, 57.8)
- added R179: 100k, Resistor_SMD:R_1206_3216Metric_Pad1.30x1.75mm_HandSolder, F.Cu at (180.2, 69.4)
- added R180: 100k, Resistor_SMD:R_1206_3216Metric_Pad1.30x1.75mm_HandSolder, F.Cu at (190.9, 69.4)
- added R181: 100k, Resistor_SMD:R_1206_3216Metric_Pad1.30x1.75mm_HandSolder, F.Cu at (180.2, 81.0)
- added R182: 100k, Resistor_SMD:R_1206_3216Metric_Pad1.30x1.75mm_HandSolder, F.Cu at (190.9, 81.0)
- added R183: 100k, Resistor_SMD:R_1206_3216Metric_Pad1.30x1.75mm_HandSolder, F.Cu at (180.2, 92.6)
- added R184: 100k, Resistor_SMD:R_1206_3216Metric_Pad1.30x1.75mm_HandSolder, F.Cu at (190.9, 92.6)
- added R185: 100k, Resistor_SMD:R_1206_3216Metric_Pad1.30x1.75mm_HandSolder, F.Cu at (180.2, 104.1)
- added R186: 100k, Resistor_SMD:R_1206_3216Metric_Pad1.30x1.75mm_HandSolder, F.Cu at (190.9, 104.1)
- added R187: 100k, Resistor_SMD:R_1206_3216Metric_Pad1.30x1.75mm_HandSolder, F.Cu at (180.2, 115.7)
- added R188: 100k, Resistor_SMD:R_1206_3216Metric_Pad1.30x1.75mm_HandSolder, F.Cu at (190.9, 115.7)
- added R189: 100k, Resistor_SMD:R_1206_3216Metric_Pad1.30x1.75mm_HandSolder, F.Cu at (180.2, 127.3)
- added R190: 100k, Resistor_SMD:R_1206_3216Metric_Pad1.30x1.75mm_HandSolder, F.Cu at (190.9, 127.3)
- added R191: 100k, Resistor_SMD:R_1206_3216Metric_Pad1.30x1.75mm_HandSolder, F.Cu at (180.2, 138.9)
- added R192: 100k, Resistor_SMD:R_1206_3216Metric_Pad1.30x1.75mm_HandSolder, F.Cu at (190.9, 138.9)
- added R2: 100k, Resistor_SMD:R_1206_3216Metric_Pad1.30x1.75mm_HandSolder, F.Cu at (233.1, 54.0)
- added R3: 100k, Resistor_SMD:R_1206_3216Metric_Pad1.30x1.75mm_HandSolder, F.Cu at (219.8, 59.9)
- C3, R20, R21, R22, R23, R24, R25, R26, R27, R44, R45, R46, R47, R48, R49, R50, R51, R68, R69, R70, R71, R72, R73, R74, R75, R92, R93, R94, R95, R96, R97, R98, R99: moved to B.Cu
- J34: value Conn_01x10 -> Conn_01x08; footprint Connector_PinHeader_2.54mm:PinHeader_1x10_P2.54mm_Vertical -> Connector_PinHeader_2.54mm:PinHeader_1x09_P2.54mm_Vertical
- J35: value Conn_01x10 -> Conn_01x08; footprint Connector_PinSocket_2.54mm:PinSocket_1x10_P2.54mm_Vertical -> Connector_PinSocket_2.54mm:PinSocket_1x08_P2.54mm_Vertical
- U2, U3, U4, U5, U6, U7, U8, U9: footprint Package_SO:SOIC-14_3.9x8.7mm_P1.27mm -> Package_DIP:DIP-14_W7.62mm_Socket_LongPads; moved to B.Cu
- moved R20 180.1 mm to (57.4, 79.5), turned to 180 degrees
- moved R21 180.1 mm to (57.4, 82.0), turned to 180 degrees
- moved R22 180.1 mm to (57.4, 84.6), turned to 180 degrees
- moved R23 180.1 mm to (57.4, 87.1), turned to 180 degrees
- moved R24 180.1 mm to (57.4, 89.7), turned to 180 degrees
- moved R25 180.1 mm to (57.4, 92.2), turned to 180 degrees
- moved R26 180.1 mm to (57.4, 94.7), turned to 180 degrees
- moved R27 180.1 mm to (57.4, 97.3), turned to 180 degrees
- moved R44 180.1 mm to (57.4, 99.8), turned to 180 degrees
- moved R45 180.1 mm to (57.4, 102.4), turned to 180 degrees
- moved R46 180.1 mm to (57.4, 104.9), turned to 180 degrees
- moved R47 180.1 mm to (57.4, 107.4), turned to 180 degrees
- moved R48 180.1 mm to (57.4, 110.0), turned to 180 degrees
- moved R49 180.1 mm to (57.4, 112.5), turned to 180 degrees
- moved R50 180.1 mm to (57.4, 115.1), turned to 180 degrees
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Connections:
- J10 pad T: /JACKS/CV_OUT_I -> Net-(J10-PadT)
- J11 pad T: /JACKS/CV_OUT_J -> Net-(J11-PadT)
- J12 pad T: /JACKS/CV_OUT_K -> Net-(J12-PadT)
- J13 pad T: /JACKS/CV_OUT_L -> Net-(J13-PadT)
- J14 pad T: /JACKS/CV_OUT_M -> Net-(J14-PadT)
- J15 pad T: /JACKS/CV_OUT_N -> Net-(J15-PadT)
- J16 pad T: /JACKS/CV_OUT_O -> Net-(J16-PadT)
- J17 pad T: /JACKS/CV_OUT_P -> Net-(J17-PadT)
- J18 pad T: /GATE_LEDs/TO_LED_A -> Net-(J18-PadT)
- J19 pad T: /GATE_LEDs/TO_LED_B -> Net-(J19-PadT)
- J2 pad T: /JACKS/CV_OUT_A -> Net-(J2-PadT)
- J20 pad T: /GATE_LEDs/TO_LED_C -> Net-(J20-PadT)
- J21 pad T: /GATE_LEDs/TO_LED_D -> Net-(J21-PadT)
- J22 pad T: /GATE_LEDs/TO_LED_E -> Net-(J22-PadT)
- J23 pad T: /GATE_LEDs/TO_LED_F -> Net-(J23-PadT)
- J24 pad T: /GATE_LEDs/TO_LED_G -> Net-(J24-PadT)
- J25 pad T: /GATE_LEDs/TO_LED_H -> Net-(J25-PadT)
- J26 pad T: /GATE_LEDs/TO_LED_I -> Net-(J26-PadT)
- J27 pad T: /GATE_LEDs/TO_LED_J -> Net-(J27-PadT)
- J28 pad T: /GATE_LEDs/TO_LED_K -> Net-(J28-PadT)
- J29 pad T: /GATE_LEDs/TO_LED_L -> Net-(J29-PadT)
- J3 pad T: /JACKS/CV_OUT_B -> Net-(J3-PadT)
- J30 pad T: /GATE_LEDs/TO_LED_M -> Net-(J30-PadT)
- J31 pad T: /GATE_LEDs/TO_LED_N -> Net-(J31-PadT)
- J32 pad T: /GATE_LEDs/TO_LED_O -> Net-(J32-PadT)
- J33 pad T: /GATE_LEDs/TO_LED_P -> Net-(J33-PadT)
- J34 pad 2: GND -> /CONTROLLER/TO_MIDI_TX
- J34 pad 3: /CONTROLLER/TO_MIDI_TX -> /CONTROLLER/FROM_MIDI_RX
- J34 pad 4: /CONTROLLER/FROM_MIDI_RX -> /CONTROLLER/SW_1
- J34 pad 5: GND -> /CONTROLLER/LED_1
- J34 pad 6: GND -> /CONTROLLER/LED_2
- J34 pad 7: /CONTROLLER/SW_1 -> GND
- J34 pad 8: /CONTROLLER/LED_1 -> +12V
- J34 pad 9: /CONTROLLER/LED_2 -> (no net)
- J35 pad 2: GND -> /MIDI/TO_MIDI_OUT
- J35 pad 3: /MIDI/TO_MIDI_OUT -> /MIDI/FROM_MIDI_IN
- J35 pad 4: /MIDI/FROM_MIDI_IN -> /IOs/FROM_SW_1
- J35 pad 5: GND -> /IOs/TO_LED_1
- J35 pad 6: GND -> /IOs/TO_LED_2
- J35 pad 7: /IOs/FROM_SW_1 -> GND
- J35 pad 8: /IOs/TO_LED_1 -> +12V
- J4 pad T: /JACKS/CV_OUT_C -> Net-(J4-PadT)
- J5 pad T: /JACKS/CV_OUT_D -> Net-(J5-PadT)
- J6 pad T: /JACKS/CV_OUT_E -> Net-(J6-PadT)
- J7 pad T: /JACKS/CV_OUT_F -> Net-(J7-PadT)
- J8 pad T: /JACKS/CV_OUT_G -> Net-(J8-PadT)
- J9 pad T: /JACKS/CV_OUT_H -> Net-(J9-PadT)
- R12 pad 2: Net-(R12-Pad2) -> /GATES/GATE_A
- R13 pad 2: Net-(R13-Pad2) -> /GATES/GATE_B
- R14 pad 2: Net-(R14-Pad2) -> /GATES/GATE_C
- R15 pad 2: Net-(R15-Pad2) -> /GATES/GATE_D
- R16 pad 2: Net-(R16-Pad2) -> /GATES/GATE_E
- R17 pad 2: Net-(R17-Pad2) -> /GATES/GATE_F
- R18 pad 2: Net-(R18-Pad2) -> /GATES/GATE_G
- R19 pad 2: Net-(R19-Pad2) -> /GATES/GATE_H
- R20 pad 1: Net-(R12-Pad2) -> Net-(J2-PadT)
- R20 pad 2: /GATES/GATE_A -> /JACKS/CV_OUT_A
- R21 pad 1: Net-(R13-Pad2) -> Net-(J3-PadT)
- R21 pad 2: /GATES/GATE_B -> /JACKS/CV_OUT_B
- R22 pad 1: Net-(R14-Pad2) -> Net-(J4-PadT)
- R22 pad 2: /GATES/GATE_C -> /JACKS/CV_OUT_C
- R23 pad 1: Net-(R15-Pad2) -> Net-(J5-PadT)
- R23 pad 2: /GATES/GATE_D -> /JACKS/CV_OUT_D
- R24 pad 1: Net-(R16-Pad2) -> Net-(J6-PadT)
- R24 pad 2: /GATES/GATE_E -> /JACKS/CV_OUT_E
- R25 pad 1: Net-(R17-Pad2) -> Net-(J7-PadT)
- R25 pad 2: /GATES/GATE_F -> /JACKS/CV_OUT_F
- R26 pad 1: Net-(R18-Pad2) -> Net-(J8-PadT)
- R26 pad 2: /GATES/GATE_G -> /JACKS/CV_OUT_G
- R27 pad 1: Net-(R19-Pad2) -> Net-(J9-PadT)
- R27 pad 2: /GATES/GATE_H -> /JACKS/CV_OUT_H
- R36 pad 2: Net-(R36-Pad2) -> /GATES/GATE_I
- R37 pad 2: Net-(R37-Pad2) -> /GATES/GATE_J
- R38 pad 2: Net-(R38-Pad2) -> /GATES/GATE_K
- R39 pad 2: Net-(R39-Pad2) -> /GATES/GATE_L
- R40 pad 2: Net-(R40-Pad2) -> /GATES/GATE_M
- R41 pad 2: Net-(R41-Pad2) -> /GATES/GATE_N
- R42 pad 2: Net-(R42-Pad2) -> /GATES/GATE_O
- R43 pad 2: Net-(R43-Pad2) -> /GATES/GATE_P
- R44 pad 1: Net-(R36-Pad2) -> Net-(J10-PadT)
- R44 pad 2: /GATES/GATE_I -> /JACKS/CV_OUT_I
- R45 pad 1: Net-(R37-Pad2) -> Net-(J11-PadT)
- R45 pad 2: /GATES/GATE_J -> /JACKS/CV_OUT_J
- R46 pad 1: Net-(R38-Pad2) -> Net-(J12-PadT)
- R46 pad 2: /GATES/GATE_K -> /JACKS/CV_OUT_K
- R47 pad 1: Net-(R39-Pad2) -> Net-(J13-PadT)
- R47 pad 2: /GATES/GATE_L -> /JACKS/CV_OUT_L
- R48 pad 1: Net-(R40-Pad2) -> Net-(J14-PadT)
- R48 pad 2: /GATES/GATE_M -> /JACKS/CV_OUT_M
- R49 pad 1: Net-(R41-Pad2) -> Net-(J15-PadT)
- R49 pad 2: /GATES/GATE_N -> /JACKS/CV_OUT_N
- R50 pad 1: Net-(R42-Pad2) -> Net-(J16-PadT)
- R50 pad 2: /GATES/GATE_O -> /JACKS/CV_OUT_O
- R51 pad 1: Net-(R43-Pad2) -> Net-(J17-PadT)
- R51 pad 2: /GATES/GATE_P -> /JACKS/CV_OUT_P
- R60 pad 2: Net-(R60-Pad2) -> /CV/CV_A
- R61 pad 2: Net-(R61-Pad2) -> /CV/CV_B
- R62 pad 2: Net-(R62-Pad2) -> /CV/CV_C
- R63 pad 2: Net-(R63-Pad2) -> /CV/CV_D
- R64 pad 2: Net-(R64-Pad2) -> /CV/CV_E
- R65 pad 2: Net-(R65-Pad2) -> /CV/CV_F
- R66 pad 2: Net-(R66-Pad2) -> /CV/CV_G
- R67 pad 2: Net-(R67-Pad2) -> /CV/CV_H
- R68 pad 1: Net-(R60-Pad2) -> Net-(J18-PadT)
- R68 pad 2: /CV/CV_A -> /GATE_LEDs/TO_LED_A
- R69 pad 1: Net-(R61-Pad2) -> Net-(J19-PadT)
- R69 pad 2: /CV/CV_B -> /GATE_LEDs/TO_LED_B
- R70 pad 1: Net-(R62-Pad2) -> Net-(J20-PadT)
- R70 pad 2: /CV/CV_C -> /GATE_LEDs/TO_LED_C
- R71 pad 1: Net-(R63-Pad2) -> Net-(J21-PadT)
- R71 pad 2: /CV/CV_D -> /GATE_LEDs/TO_LED_D
- R72 pad 1: Net-(R64-Pad2) -> Net-(J22-PadT)
- R72 pad 2: /CV/CV_E -> /GATE_LEDs/TO_LED_E
- R73 pad 1: Net-(R65-Pad2) -> Net-(J23-PadT)
- R73 pad 2: /CV/CV_F -> /GATE_LEDs/TO_LED_F
- R74 pad 1: Net-(R66-Pad2) -> Net-(J24-PadT)
- R74 pad 2: /CV/CV_G -> /GATE_LEDs/TO_LED_G
- R75 pad 1: Net-(R67-Pad2) -> Net-(J25-PadT)
- R75 pad 2: /CV/CV_H -> /GATE_LEDs/TO_LED_H
- R84 pad 2: Net-(R84-Pad2) -> /CV/CV_I
- R85 pad 2: Net-(R85-Pad2) -> /CV/CV_J
- R86 pad 2: Net-(R86-Pad2) -> /CV/CV_K
- R87 pad 2: Net-(R87-Pad2) -> /CV/CV_L
- R88 pad 2: Net-(R88-Pad2) -> /CV/CV_M
- R89 pad 2: Net-(R89-Pad2) -> /CV/CV_N
- R90 pad 2: Net-(R90-Pad2) -> /CV/CV_O
- R91 pad 2: Net-(R91-Pad2) -> /CV/CV_P
- R92 pad 1: Net-(R84-Pad2) -> Net-(J26-PadT)
- R92 pad 2: /CV/CV_I -> /GATE_LEDs/TO_LED_I
- R93 pad 1: Net-(R85-Pad2) -> Net-(J27-PadT)
- R93 pad 2: /CV/CV_J -> /GATE_LEDs/TO_LED_J
- R94 pad 1: Net-(R86-Pad2) -> Net-(J28-PadT)
- R94 pad 2: /CV/CV_K -> /GATE_LEDs/TO_LED_K
- R95 pad 1: Net-(R87-Pad2) -> Net-(J29-PadT)
- R95 pad 2: /CV/CV_L -> /GATE_LEDs/TO_LED_L
- R96 pad 1: Net-(R88-Pad2) -> Net-(J30-PadT)
- R96 pad 2: /CV/CV_M -> /GATE_LEDs/TO_LED_M
- R97 pad 1: Net-(R89-Pad2) -> Net-(J31-PadT)
- R97 pad 2: /CV/CV_N -> /GATE_LEDs/TO_LED_N
- R98 pad 1: Net-(R90-Pad2) -> Net-(J32-PadT)
- R98 pad 2: /CV/CV_O -> /GATE_LEDs/TO_LED_O
- R99 pad 1: Net-(R91-Pad2) -> Net-(J33-PadT)
- R99 pad 2: /CV/CV_P -> /GATE_LEDs/TO_LED_P
- U12 pad 1: Net-(R12-Pad2) -> /GATES/GATE_A
- U12 pad 7: Net-(R13-Pad2) -> /GATES/GATE_B
- U13 pad 1: Net-(R14-Pad2) -> /GATES/GATE_C
- U13 pad 7: Net-(R15-Pad2) -> /GATES/GATE_D
- U14 pad 1: Net-(R16-Pad2) -> /GATES/GATE_E
- U14 pad 7: Net-(R17-Pad2) -> /GATES/GATE_F
- U15 pad 1: Net-(R18-Pad2) -> /GATES/GATE_G
- U15 pad 7: Net-(R19-Pad2) -> /GATES/GATE_H
- U16 pad 1: Net-(R36-Pad2) -> /GATES/GATE_I
- U16 pad 7: Net-(R37-Pad2) -> /GATES/GATE_J
- U17 pad 1: Net-(R38-Pad2) -> /GATES/GATE_K
- U17 pad 7: Net-(R39-Pad2) -> /GATES/GATE_L
- U18 pad 1: Net-(R40-Pad2) -> /GATES/GATE_M
- U18 pad 7: Net-(R41-Pad2) -> /GATES/GATE_N
- U19 pad 1: Net-(R42-Pad2) -> /GATES/GATE_O
- U19 pad 7: Net-(R43-Pad2) -> /GATES/GATE_P
- U20 pad 1: Net-(R60-Pad2) -> /CV/CV_A
- U20 pad 7: Net-(R61-Pad2) -> /CV/CV_B
- U21 pad 1: Net-(R62-Pad2) -> /CV/CV_C
- U21 pad 7: Net-(R63-Pad2) -> /CV/CV_D
- U22 pad 1: Net-(R64-Pad2) -> /CV/CV_E
- U22 pad 7: Net-(R65-Pad2) -> /CV/CV_F
- U23 pad 1: Net-(R66-Pad2) -> /CV/CV_G
- U23 pad 7: Net-(R67-Pad2) -> /CV/CV_H
- U24 pad 1: Net-(R84-Pad2) -> /CV/CV_I
- U24 pad 7: Net-(R85-Pad2) -> /CV/CV_J
- U25 pad 1: Net-(R86-Pad2) -> /CV/CV_K
- U25 pad 7: Net-(R87-Pad2) -> /CV/CV_L
- U26 pad 1: Net-(R88-Pad2) -> /CV/CV_M
- U26 pad 7: Net-(R89-Pad2) -> /CV/CV_N
- U27 pad 1: Net-(R90-Pad2) -> /CV/CV_O
- U27 pad 7: Net-(R91-Pad2) -> /CV/CV_P
