File: mici_cv_gate_ios.kicad_sch (KiCad schematic)
At the start: 12 parts, among them Q1 2N3906, Q2 2N3906, SW1 SW_SPST

Commit message: Fixed alignment of jacks and LEDs
Parts:
- renumbered D6 to D205, D8 to D206, Q1 to Q204, Q2 to Q205, R104 to R313, R111 to R314, R110 to R315, R101 to R316, R100 to R317, R102 to R322, R103 to R323, SW1 to SW200
Changed lines of the file:
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@@
   (symbol (lib_id "Device:LED") (at 163.83 113.03 90) (unit 1)
     (in_bom yes) (on_board yes)
-    (property "Reference" "D8" (id 0) (at 166.8272 112.0394 90)
+    (property "Reference" "D206" (id 0) (at 166.8272 112.0394 90)
       (effects (font (size 1.27 1.27)) (justify right))
     )
@@
   (symbol (lib_id "Transistor_BJT:2N3906") (at 151.13 114.3 0) (mirror x) (unit 1)
     (in_bom yes) (on_board yes)
-    (property "Reference" "Q2" (id 0) (at 155.956 115.4684 0)
+    (property "Reference" "Q205" (id 0) (at 155.956 115.4684 0)
       (effects (font (size 1.27 1.27)) (justify left))
     )
@@
   (symbol (lib_id "Device:R") (at 163.83 60.96 0) (unit 1)
     (in_bom yes) (on_board yes)
-    (property "Reference" "R110" (id 0) (at 165.608 59.7916 0)
+    (property "Reference" "R315" (id 0) (at 165.608 59.7916 0)
       (effects (font (size 1.27 1.27)) (justify left))
     )
@@
   (symbol (lib_id "Device:R") (at 143.51 77.47 0) (unit 1)
     (in_bom yes) (on_board yes)
-    (property "Reference" "R102" (id 0) (at 145.288 76.3016 0)
+    (property "Reference" "R322" (id 0) (at 145.288 76.3016 0)
       (effects (font (size 1.27 1.27)) (justify left))
     )
@@
   (symbol (lib_id "Device:R") (at 138.43 114.3 270) (unit 1)
     (in_bom yes) (on_board yes)
-    (property "Reference" "R101" (id 0) (at 138.43 109.0422 90))
+    (property "Reference" "R316" (id 0) (at 138.43 109.0422 90))
     (property "Value" "100k" (id 1) (at 138.43 111.3536 90))
     (property "Footprint" "Resistor_SMD:R_1206_3216Metric_Pad1.30x1.75mm_HandSolder" (id 2) (at 138.43 112.522 90)
@@
   (symbol (lib_id "Device:LED") (at 163.83 71.12 90) (unit 1)
     (in_bom yes) (on_board yes)
-    (property "Reference" "D6" (id 0) (at 166.8272 70.1294 90)
+    (property "Reference" "D205" (id 0) (at 166.8272 70.1294 90)
       (effects (font (size 1.27 1.27)) (justify right))
     )
@@
   (symbol (lib_id "Device:R") (at 138.43 72.39 270) (unit 1)
     (in_bom yes) (on_board yes)
-    (property "Reference" "R100" (id 0) (at 138.43 67.1322 90))
+    (property "Reference" "R317" (id 0) (at 138.43 67.1322 90))
     (property "Value" "100k" (id 1) (at 138.43 69.4436 90))
     (property "Footprint" "Resistor_SMD:R_1206_3216Metric_Pad1.30x1.75mm_HandSolder" (id 2) (at 138.43 70.612 90)
@@
   (symbol (lib_id "Transistor_BJT:2N3906") (at 151.13 72.39 0) (mirror x) (unit 1)
     (in_bom yes) (on_board yes)
-    (property "Reference" "Q1" (id 0) (at 155.956 73.5584 0)
+    (property "Reference" "Q204" (id 0) (at 155.956 73.5584 0)
       (effects (font (size 1.27 1.27)) (justify left))
     )
@@
   (symbol (lib_id "Device:R") (at 163.83 102.87 0) (unit 1)
     (in_bom yes) (on_board yes)
-    (property "Reference" "R111" (id 0) (at 165.608 101.7016 0)
+    (property "Reference" "R314" (id 0) (at 165.608 101.7016 0)
       (effects (font (size 1.27 1.27)) (justify left))
     )
@@
   (symbol (lib_id "Device:R") (at 143.51 119.38 0) (unit 1)
     (in_bom yes) (on_board yes)
-    (property "Reference" "R103" (id 0) (at 145.288 118.2116 0)
+    (property "Reference" "R323" (id 0) (at 145.288 118.2116 0)
       (effects (font (size 1.27 1.27)) (justify left))
     )
@@
   (symbol (lib_id "Device:R") (at 146.05 144.78 0) (unit 1)
     (in_bom yes) (on_board yes) (fields_autoplaced)
-    (property "Reference" "R104" (id 0) (at 147.828 143.8715 0)
+    (property "Reference" "R313" (id 0) (at 147.828 143.8715 0)
       (effects (font (size 1.27 1.27)) (justify left))
     )
@@
   (symbol (lib_id "Switch:SW_SPST") (at 158.75 140.97 0) (unit 1)
     (in_bom yes) (on_board yes) (fields_autoplaced)
-    (property "Reference" "SW1" (id 0) (at 158.75 135.3525 0))
+    (property "Reference" "SW200" (id 0) (at 158.75 135.3525 0))
     (property "Value" "SW_SPST" (id 1) (at 158.75 138.1276 0))
     (property "Footprint" "My Stuff:SW_PS1024ALRED" (id 2) (at 158.75 140.97 0)

Commit message: Cleanups and title blocks
Other:
- company: (none) -> RobotDialogs
- title: (none) -> Eurorack MIDI 16x16 CV Gate
Changed lines of the file:
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@@
 (kicad_sch (version 20211123) (generator eeschema)
   (paper "A4")
+  (title_block
+    (title "Eurorack MIDI 16x16 CV Gate")
+    (date "2022-05-14")
+    (rev "1.0")
+    (company "RobotDialogs")
+  )
   (junction (at 143.51 114.3) (diameter 0) (color 0 0 0 0)
   )
