File: midi_cv_gate_dac_a.kicad_sch (KiCad schematic)
At the start: 18 parts, among them U2 MCP4922-ESL, U3 MCP4922-ESL, U4 MCP4922-ESL, U5 MCP4922-ESL, U6 MCP4922-ESL, U7 MCP4922-ESL, U8 MCP4922-ESL, U9 MCP4922-ESL

Commit message: Replace soic-14 with dip 14 for DACs, add pulldowns on opamp inputs
Parts:
- U2, U3, U4, U5, U6, U7, U8, U9: footprint Package_SO:SOIC-14_3.9x8.7mm_P1.27mm -> Package_DIP:DIP-14_W7.62mm_Socket_LongPads
Changed lines of the file:
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@@
     (property "Reference" "U7" (id 0) (at 157.5957 67.6867 0))
     (property "Value" "MCP4922-ESL" (id 1) (at 157.5957 70.4618 0))
-    (property "Footprint" "Package_SO:SOIC-14_3.9x8.7mm_P1.27mm" (id 2) (at 134.62 78.74 0)
+    (property "Footprint" "Package_DIP:DIP-14_W7.62mm_Socket_LongPads" (id 2) (at 134.62 78.74 0)
       (effects (font (size 1.27 1.27) italic) hide)
     )
@@
     (property "Reference" "U4" (id 0) (at 89.0157 103.2467 0))
     (property "Value" "MCP4922-ESL" (id 1) (at 89.0157 106.0218 0))
-    (property "Footprint" "Package_SO:SOIC-14_3.9x8.7mm_P1.27mm" (id 2) (at 66.04 114.3 0)
+    (property "Footprint" "Package_DIP:DIP-14_W7.62mm_Socket_LongPads" (id 2) (at 66.04 114.3 0)
       (effects (font (size 1.27 1.27) italic) hide)
     )
@@
     (property "Reference" "U8" (id 0) (at 157.5957 103.2467 0))
     (property "Value" "MCP4922-ESL" (id 1) (at 157.5957 106.0218 0))
-    (property "Footprint" "Package_SO:SOIC-14_3.9x8.7mm_P1.27mm" (id 2) (at 134.62 114.3 0)
+    (property "Footprint" "Package_DIP:DIP-14_W7.62mm_Socket_LongPads" (id 2) (at 134.62 114.3 0)
       (effects (font (size 1.27 1.27) italic) hide)
     )
@@
     (property "Reference" "U9" (id 0) (at 157.5957 138.8067 0))
     (property "Value" "MCP4922-ESL" (id 1) (at 157.5957 141.5818 0))
-    (property "Footprint" "Package_SO:SOIC-14_3.9x8.7mm_P1.27mm" (id 2) (at 134.62 149.86 0)
+    (property "Footprint" "Package_DIP:DIP-14_W7.62mm_Socket_LongPads" (id 2) (at 134.62 149.86 0)
       (effects (font (size 1.27 1.27) italic) hide)
     )
@@
     (property "Reference" "U2" (id 0) (at 89.0157 32.1267 0))
     (property "Value" "MCP4922-ESL" (id 1) (at 89.0157 34.9018 0))
-    (property "Footprint" "Package_SO:SOIC-14_3.9x8.7mm_P1.27mm" (id 2) (at 66.04 43.18 0)
+    (property "Footprint" "Package_DIP:DIP-14_W7.62mm_Socket_LongPads" (id 2) (at 66.04 43.18 0)
       (effects (font (size 1.27 1.27) italic) hide)
     )
@@
     (property "Reference" "U6" (id 0) (at 157.5957 32.1267 0))
     (property "Value" "MCP4922-ESL" (id 1) (at 157.5957 34.9018 0))
-    (property "Footprint" "Package_SO:SOIC-14_3.9x8.7mm_P1.27mm" (id 2) (at 134.62 43.18 0)
+    (property "Footprint" "Package_DIP:DIP-14_W7.62mm_Socket_LongPads" (id 2) (at 134.62 43.18 0)
       (effects (font (size 1.27 1.27) italic) hide)
     )
@@
     (property "Reference" "U3" (id 0) (at 89.0157 67.6867 0))
     (property "Value" "MCP4922-ESL" (id 1) (at 89.0157 70.4618 0))
-    (property "Footprint" "Package_SO:SOIC-14_3.9x8.7mm_P1.27mm" (id 2) (at 66.04 78.74 0)
+    (property "Footprint" "Package_DIP:DIP-14_W7.62mm_Socket_LongPads" (id 2) (at 66.04 78.74 0)
       (effects (font (size 1.27 1.27) italic) hide)
     )
@@
     (property "Reference" "U5" (id 0) (at 89.0157 138.8067 0))
     (property "Value" "MCP4922-ESL" (id 1) (at 89.0157 141.5818 0))
-    (property "Footprint" "Package_SO:SOIC-14_3.9x8.7mm_P1.27mm" (id 2) (at 66.04 149.86 0)
+    (property "Footprint" "Package_DIP:DIP-14_W7.62mm_Socket_LongPads" (id 2) (at 66.04 149.86 0)
       (effects (font (size 1.27 1.27) italic) hide)
     )

Commit message: Fixed alignment of jacks and LEDs
Parts:
- renumbered C9 to C14, C10 to C19, C7 to C2, C11 to C25, C12 to C30, C13 to C35, C14 to C41, R161 to R183, R160 to R186, U2 to U101, U3 to U104, U4 to U108, U5 to U111, U6 to U114, U7 to U117, U8 to U120, U9 to U123
Changed lines of the file:
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@@
   (symbol (lib_id "Analog_DAC:MCP4922-ESL") (at 134.62 78.74 0) (unit 1)
     (in_bom yes) (on_board yes) (fields_autoplaced)
-    (property "Reference" "U7" (id 0) (at 157.5957 67.6867 0))
+    (property "Reference" "U117" (id 0) (at 157.5957 67.6867 0))
     (property "Value" "MCP4922-ESL" (id 1) (at 157.5957 70.4618 0))
     (property "Footprint" "Package_DIP:DIP-14_W7.62mm_Socket_LongPads" (id 2) (at 134.62 78.74 0)
@@
   (symbol (lib_id "Device:R") (at 21.59 54.61 180) (unit 1)
     (in_bom yes) (on_board yes) (fields_autoplaced)
-    (property "Reference" "R160" (id 0) (at 23.368 53.7015 0)
+    (property "Reference" "R186" (id 0) (at 23.368 53.7015 0)
       (effects (font (size 1.27 1.27)) (justify right))
     )
@@
   (symbol (lib_id "Analog_DAC:MCP4922-ESL") (at 66.04 114.3 0) (unit 1)
     (in_bom yes) (on_board yes) (fields_autoplaced)
-    (property "Reference" "U4" (id 0) (at 89.0157 103.2467 0))
+    (property "Reference" "U108" (id 0) (at 89.0157 103.2467 0))
     (property "Value" "MCP4922-ESL" (id 1) (at 89.0157 106.0218 0))
     (property "Footprint" "Package_DIP:DIP-14_W7.62mm_Socket_LongPads" (id 2) (at 66.04 114.3 0)
@@
   (symbol (lib_id "Analog_DAC:MCP4922-ESL") (at 134.62 114.3 0) (unit 1)
     (in_bom yes) (on_board yes) (fields_autoplaced)
-    (property "Reference" "U8" (id 0) (at 157.5957 103.2467 0))
+    (property "Reference" "U120" (id 0) (at 157.5957 103.2467 0))
     (property "Value" "MCP4922-ESL" (id 1) (at 157.5957 106.0218 0))
     (property "Footprint" "Package_DIP:DIP-14_W7.62mm_Socket_LongPads" (id 2) (at 134.62 114.3 0)
@@
   (symbol (lib_id "Device:C") (at 49.53 137.16 90) (unit 1)
     (in_bom yes) (on_board yes) (fields_autoplaced)
-    (property "Reference" "C10" (id 0) (at 49.53 131.0345 90))
+    (property "Reference" "C19" (id 0) (at 49.53 131.0345 90))
     (property "Value" "100nF" (id 1) (at 49.53 133.8096 90))
     (property "Footprint" "Capacitor_SMD:C_1206_3216Metric_Pad1.33x1.80mm_HandSolder" (id 2) (at 53.34 136.1948 0)
@@
   (symbol (lib_id "Device:C") (at 49.53 30.48 90) (unit 1)
     (in_bom yes) (on_board yes) (fields_autoplaced)
-    (property "Reference" "C7" (id 0) (at 49.53 24.3545 90))
+    (property "Reference" "C2" (id 0) (at 49.53 24.3545 90))
     (property "Value" "100nF" (id 1) (at 49.53 27.1296 90))
     (property "Footprint" "Capacitor_SMD:C_1206_3216Metric_Pad1.33x1.80mm_HandSolder" (id 2) (at 53.34 29.5148 0)
@@
   (symbol (lib_id "Analog_DAC:MCP4922-ESL") (at 134.62 149.86 0) (unit 1)
     (in_bom yes) (on_board yes) (fields_autoplaced)
-    (property "Reference" "U9" (id 0) (at 157.5957 138.8067 0))
+    (property "Reference" "U123" (id 0) (at 157.5957 138.8067 0))
     (property "Value" "MCP4922-ESL" (id 1) (at 157.5957 141.5818 0))
     (property "Footprint" "Package_DIP:DIP-14_W7.62mm_Socket_LongPads" (id 2) (at 134.62 149.86 0)
@@
   (symbol (lib_id "Device:C") (at 118.11 30.48 90) (unit 1)
     (in_bom yes) (on_board yes) (fields_autoplaced)
-    (property "Reference" "C11" (id 0) (at 118.11 24.3545 90))
+    (property "Reference" "C25" (id 0) (at 118.11 24.3545 90))
     (property "Value" "100nF" (id 1) (at 118.11 27.1296 90))
     (property "Footprint" "Capacitor_SMD:C_1206_3216Metric_Pad1.33x1.80mm_HandSolder" (id 2) (at 121.92 29.5148 0)
@@
   (symbol (lib_id "Device:C") (at 49.53 101.6 90) (unit 1)
     (in_bom yes) (on_board yes) (fields_autoplaced)
-    (property "Reference" "C9" (id 0) (at 49.53 95.4745 90))
+    (property "Reference" "C14" (id 0) (at 49.53 95.4745 90))
     (property "Value" "100nF" (id 1) (at 49.53 98.2496 90))
     (property "Footprint" "Capacitor_SMD:C_1206_3216Metric_Pad1.33x1.80mm_HandSolder" (id 2) (at 53.34 100.6348 0)
@@
   (symbol (lib_id "Device:C") (at 118.11 66.04 90) (unit 1)
     (in_bom yes) (on_board yes) (fields_autoplaced)
-    (property "Reference" "C12" (id 0) (at 118.11 59.9145 90))
+    (property "Reference" "C30" (id 0) (at 118.11 59.9145 90))
     (property "Value" "100nF" (id 1) (at 118.11 62.6896 90))
     (property "Footprint" "Capacitor_SMD:C_1206_3216Metric_Pad1.33x1.80mm_HandSolder" (id 2) (at 121.92 65.0748 0)
@@
   (symbol (lib_id "Analog_DAC:MCP4922-ESL") (at 66.04 43.18 0) (unit 1)
     (in_bom yes) (on_board yes) (fields_autoplaced)
-    (property "Reference" "U2" (id 0) (at 89.0157 32.1267 0))
+    (property "Reference" "U101" (id 0) (at 89.0157 32.1267 0))
     (property "Value" "MCP4922-ESL" (id 1) (at 89.0157 34.9018 0))
     (property "Footprint" "Package_DIP:DIP-14_W7.62mm_Socket_LongPads" (id 2) (at 66.04 43.18 0)
@@
   (symbol (lib_id "Analog_DAC:MCP4922-ESL") (at 134.62 43.18 0) (unit 1)
     (in_bom yes) (on_board yes) (fields_autoplaced)
-    (property "Reference" "U6" (id 0) (at 157.5957 32.1267 0))
+    (property "Reference" "U114" (id 0) (at 157.5957 32.1267 0))
     (property "Value" "MCP4922-ESL" (id 1) (at 157.5957 34.9018 0))
     (property "Footprint" "Package_DIP:DIP-14_W7.62mm_Socket_LongPads" (id 2) (at 134.62 43.18 0)
@@
   (symbol (lib_id "Device:R") (at 24.13 54.61 180) (unit 1)
     (in_bom yes) (on_board yes) (fields_autoplaced)
-    (property "Reference" "R161" (id 0) (at 25.908 53.7015 0)
+    (property "Reference" "R183" (id 0) (at 25.908 53.7015 0)
       (effects (font (size 1.27 1.27)) (justify right))
     )
@@
   (symbol (lib_id "Analog_DAC:MCP4922-ESL") (at 66.04 78.74 0) (unit 1)
     (in_bom yes) (on_board yes) (fields_autoplaced)
-    (property "Reference" "U3" (id 0) (at 89.0157 67.6867 0))
+    (property "Reference" "U104" (id 0) (at 89.0157 67.6867 0))
     (property "Value" "MCP4922-ESL" (id 1) (at 89.0157 70.4618 0))
     (property "Footprint" "Package_DIP:DIP-14_W7.62mm_Socket_LongPads" (id 2) (at 66.04 78.74 0)
@@
   (symbol (lib_id "Device:C") (at 118.11 101.6 90) (unit 1)
     (in_bom yes) (on_board yes) (fields_autoplaced)
-    (property "Reference" "C13" (id 0) (at 118.11 95.4745 90))
+    (property "Reference" "C35" (id 0) (at 118.11 95.4745 90))
     (property "Value" "100nF" (id 1) (at 118.11 98.2496 90))
     (property "Footprint" "Capacitor_SMD:C_1206_3216Metric_Pad1.33x1.80mm_HandSolder" (id 2) (at 121.92 100.6348 0)
@@
   (symbol (lib_id "Device:C") (at 118.11 137.16 90) (unit 1)
     (in_bom yes) (on_board yes) (fields_autoplaced)
-    (property "Reference" "C14" (id 0) (at 118.11 131.0345 90))
+    (property "Reference" "C41" (id 0) (at 118.11 131.0345 90))
     (property "Value" "100nF" (id 1) (at 118.11 133.8096 90))
     (property "Footprint" "Capacitor_SMD:C_1206_3216Metric_Pad1.33x1.80mm_HandSolder" (id 2) (at 121.92 136.1948 0)
@@
   (symbol (lib_id "Analog_DAC:MCP4922-ESL") (at 66.04 149.86 0) (unit 1)
     (in_bom yes) (on_board yes) (fields_autoplaced)
-    (property "Reference" "U5" (id 0) (at 89.0157 138.8067 0))
+    (property "Reference" "U111" (id 0) (at 89.0157 138.8067 0))
     (property "Value" "MCP4922-ESL" (id 1) (at 89.0157 141.5818 0))
     (property "Footprint" "Package_DIP:DIP-14_W7.62mm_Socket_LongPads" (id 2) (at 66.04 149.86 0)

Commit message: Cleanups and title blocks
Parts:
- renumbered R183 to R92, R186 to R95
Connections:
- net CS_A renamed ~{CS_A}
- net CS_B renamed ~{CS_B}
- net CS_C renamed ~{CS_C}
- net CS_D renamed ~{CS_D}
- net CS_E renamed ~{CS_E}
- net CS_F renamed ~{CS_F}
- net CS_G renamed ~{CS_G}
- net CS_H renamed ~{CS_H}
Other:
- company: (none) -> RobotDialogs
- title: (none) -> Eurorack MIDI 16x16 CV Gate
- moved on the sheet: C14, C19, C2, C25, C30, C35, C41, C8, R92, R95, U101, U104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
