File: midi_cv_gate_midi_io.kicad_sch (KiCad schematic)
At the start: 15 parts, among them J38 DIN-5_180degree, J39 MIDI OUT, J40 DIN-5_180degree, J41 MIDI IN, U30 6N138

Commit message: Removed midi jumpers and rearranging for routing
Parts:
- removed J38, J40: DIN-5_180degree, Connector_PinSocket_2.54mm:PinSocket_1x05_P2.54mm_Vertical, symbol Connector:DIN-5_180degree
- removed JP3, JP4, JP5, JP6: SolderJumper_2_Open, Connector_PinHeader_2.54mm:PinHeader_1x02_P2.54mm_Vertical, symbol Jumper:SolderJumper_2_Open
Connections:
- net +5V: now also R108.1
- net TO_MIDI_OUT: now also R107.1
- net at D7.2 (A), U30.3 (C2): now also J41.R
- net at J41.T: now also R109.2
- no-connect marks 6 -> 1
Other:
- note removed: "For 5V: R10 = 220 R1 = 220 For 3.3V: R10 = 33 R1 = 10"
- moved on the sheet: J39, J41, R107, R108

Commit message: Fixed alignment of jacks and LEDs
Parts:
- renumbered D7 to D215, J39 to J225, J41 to J230, R108 to R372, R107 to R373, R1 to R374, R105 to R386, R109 to R388, U30 to U201
Changed lines of the file:
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@@
   (symbol (lib_id "Device:D") (at 160.02 102.87 90) (unit 1)
     (in_bom yes) (on_board yes)
-    (property "Reference" "D7" (id 0) (at 162.052 101.9615 90)
+    (property "Reference" "D215" (id 0) (at 162.052 101.9615 90)
       (effects (font (size 1.27 1.27)) (justify right))
     )
@@
   (symbol (lib_id "Connector:AudioJack3") (at 182.88 101.6 0) (mirror y) (unit 1)
     (in_bom yes) (on_board yes) (fields_autoplaced)
-    (property "Reference" "J41" (id 0) (at 189.992 101.3265 0)
+    (property "Reference" "J230" (id 0) (at 189.992 101.3265 0)
       (effects (font (size 1.27 1.27)) (justify right))
     )
@@
   (symbol (lib_id "Device:R") (at 160.02 71.12 90) (unit 1)
     (in_bom yes) (on_board yes) (fields_autoplaced)
-    (property "Reference" "R107" (id 0) (at 160.02 66.1375 90))
+    (property "Reference" "R373" (id 0) (at 160.02 66.1375 90))
     (property "Value" "220" (id 1) (at 160.02 68.9126 90))
     (property "Footprint" "Resistor_SMD:R_1206_3216Metric_Pad1.30x1.75mm_HandSolder" (id 2) (at 160.02 72.898 90)
@@
   (symbol (lib_id "Device:R") (at 168.91 106.68 90) (unit 1)
     (in_bom yes) (on_board yes) (fields_autoplaced)
-    (property "Reference" "R109" (id 0) (at 168.91 101.6975 90))
+    (property "Reference" "R388" (id 0) (at 168.91 101.6975 90))
     (property "Value" "220" (id 1) (at 168.91 104.4726 90))
     (property "Footprint" "Resistor_SMD:R_1206_3216Metric_Pad1.30x1.75mm_HandSolder" (id 2) (at 168.91 108.458 90)
@@
   (symbol (lib_id "Connector:AudioJack3") (at 172.72 71.12 180) (unit 1)
     (in_bom yes) (on_board yes) (fields_autoplaced)
-    (property "Reference" "J39" (id 0) (at 179.832 69.5765 0)
+    (property "Reference" "J225" (id 0) (at 179.832 69.5765 0)
       (effects (font (size 1.27 1.27)) (justify right))
     )
@@
   (symbol (lib_id "Device:R") (at 137.16 113.03 0) (unit 1)
     (in_bom yes) (on_board yes) (fields_autoplaced)
-    (property "Reference" "R1" (id 0) (at 138.938 112.1215 0)
+    (property "Reference" "R374" (id 0) (at 138.938 112.1215 0)
       (effects (font (size 1.27 1.27)) (justify left))
     )
@@
   (symbol (lib_id "Device:R") (at 129.54 102.87 0) (unit 1)
     (in_bom yes) (on_board yes) (fields_autoplaced)
-    (property "Reference" "R105" (id 0) (at 131.318 101.9615 0)
+    (property "Reference" "R386" (id 0) (at 131.318 101.9615 0)
       (effects (font (size 1.27 1.27)) (justify left))
     )
@@
   (symbol (lib_id "Device:R") (at 152.4 68.58 90) (unit 1)
     (in_bom yes) (on_board yes) (fields_autoplaced)
-    (property "Reference" "R108" (id 0) (at 152.4 63.5975 90))
+    (property "Reference" "R372" (id 0) (at 152.4 63.5975 90))
     (property "Value" "220" (id 1) (at 152.4 66.3726 90))
     (property "Footprint" "Resistor_SMD:R_1206_3216Metric_Pad1.30x1.75mm_HandSolder" (id 2) (at 152.4 70.358 90)
@@
   (symbol (lib_id "Isolator:6N138") (at 147.32 101.6 180) (unit 1)
     (in_bom yes) (on_board yes) (fields_autoplaced)
-    (property "Reference" "U30" (id 0) (at 147.32 90.0135 0))
+    (property "Reference" "U201" (id 0) (at 147.32 90.0135 0))
     (property "Value" "6N138" (id 1) (at 147.32 92.7886 0))
     (property "Footprint" "Package_DIP:DIP-8_W7.62mm_Socket_LongPads" (id 2) (at 139.954 93.98 0)

Commit message: Cleanups and title blocks
Other:
- company: (none) -> RobotDialogs
- title: (none) -> Eurorack MIDI 16x16 CV Gate
Changed lines of the file:
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@@
 (kicad_sch (version 20211123) (generator eeschema)
   (paper "A4")
+  (title_block
+    (title "Eurorack MIDI 16x16 CV Gate")
+    (date "2022-05-14")
+    (rev "1.0")
+    (company "RobotDialogs")
+  )
   (junction (at 160.02 99.06) (diameter 0) (color 0 0 0 0)
   )
